Commit message: Added color to the robot.

File: src/my_robot/urdf/my_robot.xacro (robot description, xacro)
@@ -176,3 +176,19 @@
     <axis xyz="0 1 0" rpy="0 0 0"/>
   </joint>
+    <!-- colors  -->
+    <gazebo reference="left_wheel">
+        <material>Gazebo/Blue</material>
+    </gazebo>
+    <gazebo reference="right_wheel">
+        <material>Gazebo/Blue</material>
+    </gazebo>
+    <gazebo reference="chassis">
+        <material>Gazebo/Green</material>
+    </gazebo>
+    <gazebo reference="hokuyo">
+        <material>Gazebo/Black</material>
+    </gazebo>
+    <gazebo reference="camera">
+        <material>Gazebo/Gray</material>
+    </gazebo>
 </robot>

Commit message: Updated the .gazebo and .xacro file for sensor upgrade.

File: src/my_robot/urdf/my_robot.xacro (robot description, xacro)
@@ -176,19 +176,26 @@
     <axis xyz="0 1 0" rpy="0 0 0"/>
   </joint>
-    <!-- colors  -->
-    <gazebo reference="left_wheel">
-        <material>Gazebo/Blue</material>
-    </gazebo>
-    <gazebo reference="right_wheel">
-        <material>Gazebo/Blue</material>
-    </gazebo>
-    <gazebo reference="chassis">
-        <material>Gazebo/Green</material>
-    </gazebo>
-    <gazebo reference="hokuyo">
-        <material>Gazebo/Black</material>
-    </gazebo>
-    <gazebo reference="camera">
-        <material>Gazebo/Gray</material>
-    </gazebo>
+  <joint name="camera_optical_joint" type="fixed">
+    <origin xyz="0 0 0" rpy="-1.5707 0 -1.5707"/>
+    <parent link="camera"/>
+    <child link="camera_link_optical"/>
+  </joint>
+  <link name="camera_link_optical">
+  </link>
+  <!-- colors  -->
+  <gazebo reference="left_wheel">
+    <material>Gazebo/Blue</material>
+  </gazebo>
+  <gazebo reference="right_wheel">
+    <material>Gazebo/Blue</material>
+  </gazebo>
+  <gazebo reference="chassis">
+    <material>Gazebo/Green</material>
+  </gazebo>
+  <gazebo reference="hokuyo">
+    <material>Gazebo/Black</material>
+  </gazebo>
+  <gazebo reference="camera">
+    <material>Gazebo/Gray</material>
+  </gazebo>
 </robot>
